File: płytka_MCP_I2C_v1/płytka_MCP_I2C.kicad_pcb (KiCad board)
At the start: 2 copper layers, 98 x 77 mm, 33 parts, among them J1 A0, J10 V0, J11 Ext, J12 I2C, J13 U2, J15 U2, J16 U3, J17 RS, J18 K, J19 A, J2 A1, J20 VDD, J21 GND, J23 VSS, J24 Conn_01x16_Pin, J25 LCD, J26 VCC, J3 A2, J4 SDA, J5 SCL, J6 INTA, J7 INTB, J8 INTA, J9 RESET, U1 MCP23017_SP

Commit message: Wersja 2 plytki I2C
Parts:
- removed J13: U2, Library:PinSocket_1x08_P2.54mm_Vertical_kwadrat
- removed J9: RESET, Connector_PinSocket_2.54mm:PinSocket_1x01_P2.54mm_Vertical
- added ?: , , F.Cu at (40.6, 42.0)
- added ?: , , F.Cu at (40.5, 109.3)
- added ?: , , F.Cu at (128.8, 109.4)
- added ?: , , F.Cu at (129.3, 42.0)
- added J14: U1, Library:PinSocket_1x03_P2.54mm_Vertical, F.Cu at (60.9, 53.7)
- moved J16 22.8 mm to (44.9, 85.3), turned to 180 degrees
- moved J25 16.1 mm to (45.6, 109.3)
- moved J24 16.1 mm to (45.6, 102.2)
- moved J26 12.7 mm to (98.5, 88.7), turned to 0 degrees
- moved J19 10.3 mm to (52.1, 59.0)
- moved J18 10.3 mm to (52.1, 53.2)
- moved R1 10.1 mm to (98.2, 46.3)
- moved R6 10.1 mm to (103.8, 56.3)
- moved J21 9.80 mm to (105.0, 88.8), turned to 0 degrees
- moved R2 9.58 mm to (109.4, 46.3)
- moved R3 9.33 mm to (115.1, 46.3)
- moved J8 9.19 mm to (73.2, 53.6)
- moved J1 9.19 mm to (90.7, 49.5)
- moved J2 9.19 mm to (85.7, 49.5)
- moved J3 9.19 mm to (80.7, 49.5)
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Connections:
- U1 pad 1: Net-(J15-Pin_1) -> Net-(J14-Pin_3)
- U1 pad 2: Net-(J15-Pin_2) -> Net-(J14-Pin_2)
- U1 pad 21: Net-(J13-Pin_1) -> Net-(J15-Pin_1)
- U1 pad 22: Net-(J13-Pin_2) -> Net-(J15-Pin_2)
- U1 pad 23: Net-(J13-Pin_3) -> Net-(J15-Pin_3)
- U1 pad 24: Net-(J13-Pin_4) -> Net-(J15-Pin_4)
- U1 pad 25: Net-(J13-Pin_5) -> Net-(J15-Pin_5)
- U1 pad 26: Net-(J13-Pin_6) -> Net-(J15-Pin_6)
- U1 pad 27: Net-(J13-Pin_7) -> Net-(J15-Pin_7)
- U1 pad 28: Net-(J13-Pin_8) -> Net-(J15-Pin_8)
- U1 pad 3: Net-(J15-Pin_3) -> Net-(J14-Pin_1)
- U1 pad 4: Net-(J15-Pin_4) -> unconnected-(U1-GPB3-Pad4)
- U1 pad 5: Net-(J15-Pin_5) -> unconnected-(U1-GPB4-Pad5)
- U1 pad 6: Net-(J15-Pin_6) -> unconnected-(U1-GPB5-Pad6)
- U1 pad 7: Net-(J15-Pin_7) -> unconnected-(U1-GPB6-Pad7)
- U1 pad 8: Net-(J15-Pin_8) -> unconnected-(U1-GPB7-Pad8)
Routing:
- net VCC: track 131.3 -> 195.8 mm
- net Net-(J15-Pin_1): track 11.1 -> 54.4 mm
- net Net-(U1-~{RESET}): track 65.0 -> 23.0 mm
- net Net-(J16-Pin_7): track 25.5 -> 67.4 mm
- net GND: track 161.8 -> 121.3 mm
- net Net-(J16-Pin_8): track 33.1 -> 72.8 mm
- net Net-(J15-Pin_2): track 11.1 -> 50.1 mm
- net Net-(J13-Pin_1): track 37.9 -> 0.00 mm
- net Net-(J16-Pin_6): track 25.5 -> 62.4 mm
- net Net-(J13-Pin_2): track 34.4 -> 0.00 mm
- net Net-(J15-Pin_3): track 11.1 -> 43.1 mm
- net Net-(J16-Pin_5): track 25.5 -> 56.9 mm
- net Net-(J13-Pin_3): track 31.0 -> 0.00 mm
- net Net-(J15-Pin_4): track 11.1 -> 39.9 mm
- net Net-(J14-Pin_1): track 0.00 -> 27.6 mm
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Other:
- board text added: "P2"
