File: płytka_MCP_I2C_v1/płytka_MCP_I2C.kicad_sch (KiCad schematic)
At the start: 33 parts, among them J1 A0, J10 V0, J11 Ext, J12 I2C, J13 U2, J15 U2, J16 U3, J17 RS, J18 K, J19 A, J2 A1, J20 VDD, J21 GND, J23 VSS, J24 Conn_01x16_Pin, J25 LCD, J26 VCC, J3 A2, J4 SDA, J5 SCL, J6 INTA, J7 INTB, J8 INTA, J9 RESET, U1 MCP23017_SP

Commit message: Wersja 2 plytki I2C
Parts:
- removed J13: U2, Library:PinSocket_1x08_P2.54mm_Vertical_kwadrat, symbol Connector:Conn_01x08_Pin
- added J14: U1, Library:PinSocket_1x03_P2.54mm_Vertical, symbol Connector:Conn_01x03_Pin
Connections:
- net at J15.1 (Pin_1): now also U1.21 (GPA0); no longer U1.1 (GPB0)
- net at J15.2 (Pin_2): now also U1.22 (GPA1); no longer U1.2 (GPB1)
- net at J15.3 (Pin_3): now also U1.23 (GPA2); no longer U1.3 (GPB2)
- net at J15.4 (Pin_4): now also U1.24 (GPA3); no longer U1.4 (GPB3)
- net at J15.5 (Pin_5): now also U1.25 (GPA4); no longer U1.5 (GPB4)
- net at J15.6 (Pin_6): now also U1.26 (GPA5); no longer U1.6 (GPB5)
- net at J15.7 (Pin_7): now also U1.27 (GPA6); no longer U1.7 (GPB6)
- net at J15.8 (Pin_8): now also U1.28 (GPA7); no longer U1.8 (GPB7)
- new net: J14.1 (Pin_1), U1.3 (GPB2)
- new net: J14.2 (Pin_2), U1.2 (GPB1)
- new net: J14.3 (Pin_3), U1.1 (GPB0)
- no-connect marks 0 -> 5
Other:
- moved on the sheet: J12, J15, J8, J9
