File: płytka_MCP_SPI/płytka_MCP_I2C.kicad_pcb (KiCad board)
At the start: 2 copper layers, 98 x 77 mm, 33 parts, among them J1 A0, J10 V0, J11 Ext, J12 I2C, J13 U2, J15 U2, J16 U3, J17 RS, J18 K, J19 A, J2 A1, J20 VDD, J21 GND, J23 VSS, J24 Conn_01x16_Pin, J25 LCD, J26 VCC, J3 A2, J4 SDA, J5 SCL, J6 INTA, J7 INTB, J8 INTA, J9 RESET, U1 MCP23017_SP

Commit message: MCP_SPI płytka wersja 1.0
Parts:
- removed J12: I2C, Connector_PinSocket_2.54mm:PinSocket_1x02_P2.54mm_Vertical
- removed J4: SDA, Library:PinSocket_1x03_P2.54mm_Vertical
- removed J5: SCL, Library:PinSocket_1x03_P2.54mm_Vertical
- removed R2, R3: 4.7k, Library:R_Axial_DIN0207_L6.3mm_D2.5mm_P10.16mm_Horizontal_square
- added J27: SPI, Connector_PinSocket_2.54mm:PinSocket_1x04_P2.54mm_Vertical, F.Cu at (119.2, 78.3)
- U1: value MCP23017_SP -> MCP23S17_SP
- moved J18 35.9 mm to (61.8, 77.2)
- moved J19 35.6 mm to (61.8, 82.6)
- moved J17 19.2 mm to (61.9, 71.1), turned to 180 degrees
- moved R4 12.4 mm to (115.9, 40.3)
- moved R5 11.6 mm to (120.6, 40.3)
- moved J6 10.4 mm to (111.8, 60.6)
- moved J7 10.4 mm to (118.1, 60.6)
- moved RV1 4.15 mm to (126.5, 100.3)
- moved J13 2.38 mm to (62.0, 42.2)
- moved R6 0.88 mm to (111.1, 50.5)
Connections:
- U1 pad 11: unconnected-(U1-NC-Pad11) -> Net-(J27-Pin_4)
- U1 pad 14: unconnected-(U1-NC-Pad14) -> Net-(J27-Pin_1)
Routing:
- net Net-(J19-Pin_1): track 128.3 -> 64.4 mm
- net Net-(J18-Pin_1): track 109.4 -> 69.5 mm
- net Net-(J6-Pin_2): track 70.9 -> 46.0 mm
- net Net-(J27-Pin_1): track 0.00 -> 22.6 mm
- net Net-(J4-Pin_1): track 20.5 -> 0.00 mm
- net Net-(J5-Pin_1): track 20.2 -> 0.00 mm
- net Net-(J27-Pin_4): track 0.00 -> 19.8 mm
- net VCC: track 131.3 -> 111.8 mm
- net Net-(J17-Pin_1): track 69.7 -> 53.5 mm
- net Net-(J27-Pin_3): track 34.0 -> 21.1 mm
- net Net-(J17-Pin_3): track 61.1 -> 67.2 mm
- net Net-(J17-Pin_2): track 67.4 -> 62.1 mm
- net Net-(J7-Pin_2): track 60.9 -> 56.9 mm
- net GND: track 161.8 -> 158.2 mm
- net Net-(J10-Pin_1): track 10.5 -> 7.08 mm
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Other:
- board size 98 x 77 mm -> 77.3 x 77 mm
- board text added: "CS"
- board text added: "SCK"
- board text added: "SI"
- board text added: "SO"
- board text added: "SPI"
- board text removed: "SCL"
- board text removed: "SDA"
