File: MCP_I2C_SPI_alternatywna_V11/MCP_I2C_SPI.kicad_pcb (KiCad board)
At the start: 2 copper layers, 97.7 x 98.8 mm, 42 parts, among them J1 GPA, J10 VCC, J11 GND, J12 I2C, J13 Interrupt0, J14 A2, J15 A1, J16 A0, J17 SDA, J18 SCK, J19 INTA, J2 GPB, J20 INTB, J21 V0, J22 Ext, J23 SPI, J24 InterruptS, J25 A2, J27 GPB, J28 GPA, J29 A1, J3 Data, J31 A0, J32 INTA, J33 INTB, J4 Control, J5 Zlacze_LCD, J6 VSS, J65 SIL9, J66 SIL5, J7 K, J8 VDD, J9 A, U1 MCP23017_SP, U2 MCP23017_SP

Commit message: MCP_I2C_SPI PCB V11
Parts:
- J5: value Zlacze_LCD -> Złącze LCD
- moved RV1 1.00 mm to (144.3, 109.0)
Connections:
- J7 pad 1: Net-(J5-Pin_15) -> Net-(J5-Pin_16)
- J9 pad 1: Net-(J5-Pin_16) -> Net-(J5-Pin_15)
Routing:
- net Net-(J5-Pin_15): track 88.7 -> 110.3 mm
- net SCL: track 101.0 -> 118.7 mm
- net Net-(J5-Pin_16): track 110.0 -> 93.5 mm
- net GND: track 262.1 -> 275.8 mm, vias 1 -> 0
- net SDA: track 118.5 -> 127.9 mm
- net Net-(J2-Pin_8): track 38.2 -> 33.0 mm
- net +5V: track 318.8 -> 317.4 mm

Commit message: MCP_I2C_SPI PCB V12
Parts:
- U2: value MCP23017_SP -> MCP23S17_SP
Routing:
- net +5V: track 317.4 -> 321.1 mm
- net GND: track 275.8 -> 276.9 mm

Commit message: Final verison MCP_I2C_SPI, ready to order
Parts:
- J22: value Ext -> EXT
- moved J10 3.68 mm to (74.0, 29.8)
- moved J22 0.30 mm to (124.7, 110.7)
Routing:
- net SDA: track 127.9 -> 139.1 mm
- net SCL: track 118.7 -> 123.9 mm
- net +5V: track 321.1 -> 319.5 mm
- net Net-(J5-Pin_15): track 110.3 -> 111.2 mm
- net Net-(J5-Pin_1): track 76.3 -> 75.4 mm
- net Net-(J5-Pin_16): track 93.5 -> 94.1 mm
Other:
- board size 97.7 x 98.8 mm -> 98 x 98.8 mm
- board text added: "INT"
- board text added: "UP"
