File: MCP_I2C_SPI_alternatywna_V11/MCP_I2C_SPI.kicad_sch (KiCad schematic)
At the start: 48 parts, among them J10 VCC, J11 GND, J21 V0, J22 Ext, J26 I2C, J3 Data, J30 Interrupt0, J34 A2, J35 SDA, J36 GPB, J37 GPA, J38 A1, J39 SCK, J4 Control, J40 A0, J41 INTA, J42 INTB, J43 SPI, J44 InterruptS, J45 A2, J46 GPB, J47 GPA, J48 A1, J49 A0, J5 Zlacze_LCD, J50 INTA, J51 INTB, J6 VSS, J65 Conn_01x09_Pin, J66 SIL5, J7 K, J8 VDD, J9 A, U3 MCP23017_SP, U4 MCP23017_SP

Commit message: MCP_I2C_SPI PCB V11
Connections:
- net at J5.15 (Pin_15): now also J9.1 (Pin_1); no longer J7.1 (Pin_1)
- net at J5.16 (Pin_16): now also J7.1 (Pin_1); no longer J9.1 (Pin_1)
Changed lines of the file:
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@@
+	(wire
+		(pts
+			(xy 77.47 156.21) (xy 77.47 110.49)
+		)
+		(stroke
+			(width 0)
+			(type default)
+		)
+	)
 	(wire
 		(pts
@@
 	(wire
 		(pts
+			(xy 74.93 113.03) (xy 57.15 113.03)
+		)
+		(stroke
+			(width 0)
+			(type default)
+		)
+	)
+	(wire
+		(pts
 			(xy 43.18 83.82) (xy 43.18 86.36)
 		)
@@
 	(wire
 		(pts
-			(xy 53.34 115.57) (xy 77.47 115.57)
-		)
-		(stroke
-			(width 0)
-			(type default)
-		)
-	)
-	(wire
-		(pts
 			(xy 45.72 88.9) (xy 45.72 74.93)
 		)
@@
 	(wire
 		(pts
-			(xy 50.8 118.11) (xy 74.93 118.11)
-		)
-		(stroke
-			(width 0)
-			(type default)
-		)
-	)
-	(wire
-		(pts
 			(xy 266.7 104.14) (xy 266.7 88.9)
 		)
@@
 	(wire
 		(pts
-			(xy 50.8 93.98) (xy 50.8 118.11)
-		)
-		(stroke
-			(width 0)
-			(type default)
-		)
-	)
-	(wire
-		(pts
 			(xy 222.25 73.66) (xy 236.22 73.66)
 		)
@@
 	(wire
 		(pts
-			(xy 77.47 115.57) (xy 77.47 156.21)
-		)
-		(stroke
-			(width 0)
-			(type default)
-		)
-	)
-	(wire
-		(pts
 			(xy 264.16 93.98) (xy 265.43 93.98)
 		)
@@
 	(wire
 		(pts
+			(xy 77.47 110.49) (xy 59.69 110.49)
+		)
+		(stroke
+			(width 0)
+			(type default)
+		)
+	)
+	(wire
+		(pts
 			(xy 25.4 114.3) (xy 25.4 144.78)
 		)
@@
 	(wire
 		(pts
+			(xy 74.93 113.03) (xy 74.93 156.21)
+		)
+		(stroke
+			(width 0)
+			(type default)
+		)
+	)
+	(wire
+		(pts
 			(xy 30.48 43.18) (xy 30.48 45.72)
 		)
@@
 	(wire
 		(pts
-			(xy 74.93 118.11) (xy 74.93 156.21)
-		)
-		(stroke
-			(width 0)
-			(type default)
-		)
-	)
-	(wire
-		(pts
 			(xy 64.77 128.27) (xy 64.77 156.21)
 		)
@@
 	(wire
 		(pts
-			(xy 53.34 63.5) (xy 53.34 115.57)
-		)
-		(stroke
-			(width 0)
-			(type default)
-		)
-	)
-	(wire
-		(pts
 			(xy 226.06 62.23) (xy 226.06 71.12)
 		)
@@
 	(wire
 		(pts
+			(xy 59.69 110.49) (xy 59.69 93.98)
+		)
+		(stroke
+			(width 0)
+			(type default)
+		)
+	)
+	(wire
+		(pts
 			(xy 171.45 156.21) (xy 171.45 171.45)
 		)
@@
 	(wire
 		(pts
+			(xy 59.69 93.98) (xy 43.18 93.98)
+		)
+		(stroke
+			(width 0)
+			(type default)
+		)
+	)
+	(wire
+		(pts
 			(xy 213.36 80.01) (xy 213.36 68.58)
 		)
@@
 	(wire
 		(pts
-			(xy 43.18 93.98) (xy 50.8 93.98)
-		)
-		(stroke
-			(width 0)
-			(type default)
-		)
-	)
-	(wire
-		(pts
 			(xy 153.67 77.47) (xy 171.45 77.47)
 		)
@@
 	(wire
 		(pts
-			(xy 43.18 63.5) (xy 53.34 63.5)
-		)
-		(stroke
-			(width 0)
-			(type default)
-		)
-	)
-	(wire
-		(pts
 			(xy 160.02 133.35) (xy 171.45 133.35)
 		)
@@
 	(wire
 		(pts
+			(xy 57.15 63.5) (xy 43.18 63.5)
+		)
+		(stroke
+			(width 0)
+			(type default)
+		)
+	)
+	(wire
+		(pts
 			(xy 149.86 26.67) (xy 163.83 26.67)
 		)
@@
 		)
 		(stroke
+			(width 0)
+			(type default)
+		)
+	)
+	(wire
+		(pts
+			(xy 57.15 113.03) (xy 57.15 63.5)
+		)
+		(stroke

Commit message: Final verison MCP_I2C_SPI, ready to order
Parts:
- J65: value Conn_01x09_Pin -> SIL9
- renumbered C3 to C1, C4 to C2, J37 to J1, J26 to J12, J30 to J13, J34 to J14, J38 to J15, J40 to J16, J35 to J17, J39 to J18, J41 to J19, J36 to J2, J42 to J20, J43 to J23, J44 to J24, J45 to J25, J46 to J27, J47 to J28, J48 to J29, J49 to J31, J50 to J32, J51 to J33, U3 to U1, U4 to U2
Changed lines of the file:
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@@
 		(on_board yes)
 		(dnp no)
-		(property "Reference" "J42"
+		(property "Reference" "J20"
 			(at 172.72 44.45 0)
 			(effects
@@
 			(project "MCP_I2C_SPI"
 				(path "/6e11339b-95d5-4292-a9a2-34157a3ab292"
-					(reference "J42")
+					(reference "J20")
 					(unit 1)
 				)
@@
 		(on_board yes)
 		(dnp no)
-		(property "Reference" "J51"
+		(property "Reference" "J33"
 			(at 259.08 86.36 0)
 			(effects
@@
 			(project "MCP_I2C_SPI"
 				(path "/6e11339b-95d5-4292-a9a2-34157a3ab292"
-					(reference "J51")
+					(reference "J33")
 					(unit 1)
 				)
@@
 		(on_board yes)
 		(dnp no)
-		(property "Reference" "J44"
+		(property "Reference" "J24"
 			(at 167.894 84.582 0)
 			(effects
@@
 			(project "MCP_I2C_SPI"
 				(path "/6e11339b-95d5-4292-a9a2-34157a3ab292"
-					(reference "J44")
+					(reference "J24")
 					(unit 1)
 				)
@@
 		(on_board yes)
 		(dnp no)
-		(property "Reference" "J35"
+		(property "Reference" "J17"
 			(at 130.81 44.45 0)
 			(effects
@@
 			(project "MCP_I2C_SPI"
 				(path "/6e11339b-95d5-4292-a9a2-34157a3ab292"
-					(reference "J35")
+					(reference "J17")
 					(unit 1)
 				)
@@
 		(on_board yes)
 		(dnp no)
-		(property "Reference" "J48"
+		(property "Reference" "J29"
 			(at 231.14 66.04 0)
 			(effects
@@
 			(project "MCP_I2C_SPI"
 				(path "/6e11339b-95d5-4292-a9a2-34157a3ab292"
-					(reference "J48")
+					(reference "J29")
 					(unit 1)
 				)
@@
 		(dnp no)
 		(fields_autoplaced yes)
-		(property "Reference" "C4"
+		(property "Reference" "C2"
 			(at 185.42 97.79 90)
 			(effects
@@
 			(project "MCP_I2C_SPI"
 				(path "/6e11339b-95d5-4292-a9a2-34157a3ab292"
-					(reference "C4")
+					(reference "C2")
 					(unit 1)
 				)
@@
 		(on_board yes)
 		(dnp no)
-		(property "Reference" "J36"
+		(property "Reference" "J2"
 			(at 136.144 80.518 0)
 			(effects
@@
 			(project "MCP_I2C_SPI"
 				(path "/6e11339b-95d5-4292-a9a2-34157a3ab292"
-					(reference "J36")
+					(reference "J2")
 					(unit 1)
 				)
@@
 		(dnp no)
 		(fields_autoplaced yes)
-		(property "Reference" "J37"
+		(property "Reference" "J1"
 			(at 133.35 104.1399 0)
 			(effects
@@
 			(project "MCP_I2C_SPI"
 				(path "/6e11339b-95d5-4292-a9a2-34157a3ab292"
-					(reference "J37")
+					(reference "J1")
 					(unit 1)
 				)
@@
 		(on_board yes)
 		(dnp no)
-		(property "Reference" "J45"
+		(property "Reference" "J25"
 			(at 217.17 66.04 0)
 			(effects
@@
 			(project "MCP_I2C_SPI"
 				(path "/6e11339b-95d5-4292-a9a2-34157a3ab292"
-					(reference "J45")
+					(reference "J25")
 					(unit 1)
 				)
@@
 		(on_board yes)
 		(dnp no)
-		(property "Reference" "J50"
+		(property "Reference" "J32"
 			(at 245.11 86.36 0)
 			(effects
@@
 			(project "MCP_I2C_SPI"
 				(path "/6e11339b-95d5-4292-a9a2-34157a3ab292"
-					(reference "J50")
+					(reference "J32")
 					(unit 1)
 				)
@@
 		(on_board yes)
 		(dnp no)
-		(property "Reference" "J30"
+		(property "Reference" "J13"
 			(at 81.026 42.926 0)
 			(effects
@@
 			(project "MCP_I2C_SPI"
 				(path "/6e11339b-95d5-4292-a9a2-34157a3ab292"
-					(reference "J30")
+					(reference "J13")
 					(unit 1)
 				)
@@
 			)
 		)
-		(property "Value" "Conn_01x09_Pin"
+		(property "Value" "SIL9"
 			(at 59.055 16.51 0)
 			(effects
@@
 		(on_board yes)
 		(dnp no)
-		(property "Reference" "J39"
+		(property "Reference" "J18"
 			(at 144.78 44.45 0)
 			(effects
@@
 			(project "MCP_I2C_SPI"
 				(path "/6e11339b-95d5-4292-a9a2-34157a3ab292"
-					(reference "J39")
+					(reference "J18")
 					(unit 1)
 				)
@@
 		(on_board yes)
 		(dnp no)
-		(property "Reference" "J40"
+		(property "Reference" "J16"
 			(at 158.75 24.13 0)
 			(effects
@@
 			(project "MCP_I2C_SPI"
 				(path "/6e11339b-95d5-4292-a9a2-34157a3ab292"
-					(reference "J40")
+					(reference "J16")
 					(unit 1)
 				)
@@
 		(dnp no)
 		(fields_autoplaced yes)
-		(property "Reference" "U4"
+		(property "Reference" "U2"
 			(at 191.3733 107.95 0)
 			(effects
@@
 			(project "MCP_I2C_SPI"
 				(path "/6e11339b-95d5-4292-a9a2-34157a3ab292"
-					(reference "U4")
+					(reference "U2")
 					(unit 1)
 				)
@@
 		(dnp no)
 		(fields_autoplaced yes)
-		(property "Reference" "U3"
+		(property "Reference" "U1"
 			(at 105.0133 66.04 0)
 			(effects
@@
 			(project "MCP_I2C_SPI"
 				(path "/6e11339b-95d5-4292-a9a2-34157a3ab292"
-					(reference "U3")
+					(reference "U1")
 					(unit 1)
 				)
@@
 		(on_board yes)
 		(dnp no)
-		(property "Reference" "J46"
+		(property "Reference" "J27"
 			(at 222.504 122.428 0)
 			(effects
@@
 			(project "MCP_I2C_SPI"
 				(path "/6e11339b-95d5-4292-a9a2-34157a3ab292"
-					(reference "J46")
+					(reference "J27")
 					(unit 1)
 				)
@@
 		(dnp no)
 		(fields_autoplaced yes)
-		(property "Reference" "C3"
+		(property "Reference" "C1"
 			(at 99.06 55.88 90)
 			(effects
@@
 			(project "MCP_I2C_SPI"
 				(path "/6e11339b-95d5-4292-a9a2-34157a3ab292"
-					(reference "C3")
+					(reference "C1")
 					(unit 1)
 				)
@@
 		(dnp no)
 		(fields_autoplaced yes)
-		(property "Reference" "J47"
+		(property "Reference" "J28"
 			(at 219.71 146.0499 0)
 			(effects
@@
 			(project "MCP_I2C_SPI"
 				(path "/6e11339b-95d5-4292-a9a2-34157a3ab292"
-					(reference "J47")
+					(reference "J28")
 					(unit 1)
 				)
@@
 		(on_board yes)
 		(dnp no)
-		(property "Reference" "J38"
+		(property "Reference" "J15"
 			(at 144.78 24.13 0)
 			(effects
@@
 			(project "MCP_I2C_SPI"
 				(path "/6e11339b-95d5-4292-a9a2-34157a3ab292"
-					(reference "J38")
+					(reference "J15")
 					(unit 1)
 				)
@@
 		(on_board yes)
 		(dnp no)
-		(property "Reference" "J26"
+		(property "Reference" "J12"
 			(at 80.264 33.782 0)
 			(effects
@@
 			(project "MCP_I2C_SPI"
 				(path "/6e11339b-95d5-4292-a9a2-34157a3ab292"
-					(reference "J26")
+					(reference "J12")
 					(unit 1)
 				)
@@
 		(on_board yes)
 		(dnp no)
-		(property "Reference" "J43"
+		(property "Reference" "J23"
 			(at 166.624 70.866 0)
 			(effects
@@
 			(project "MCP_I2C_SPI"
 				(path "/6e11339b-95d5-4292-a9a2-34157a3ab292"
-					(reference "J43")
+					(reference "J23")
 					(unit 1)
 				)
@@
 		(on_board yes)
 		(dnp no)
-		(property "Reference" "J41"
+		(property "Reference" "J19"
 			(at 158.75 44.45 0)
 			(effects
@@
 			(project "MCP_I2C_SPI"
 				(path "/6e11339b-95d5-4292-a9a2-34157a3ab292"
-					(reference "J41")
+					(reference "J19")
 					(unit 1)
 				)
@@
 		(on_board yes)
 		(dnp no)
-		(property "Reference" "J34"
+		(property "Reference" "J14"
 			(at 130.81 24.13 0)
 			(effects
@@
 			(project "MCP_I2C_SPI"
 				(path "/6e11339b-95d5-4292-a9a2-34157a3ab292"
-					(reference "J34")
+					(reference "J14")
 					(unit 1)
 				)
@@
 		(on_board yes)
 		(dnp no)
-		(property "Reference" "J49"
+		(property "Reference" "J31"
 			(at 245.11 66.04 0)
 			(effects
@@
 			(project "MCP_I2C_SPI"
 				(path "/6e11339b-95d5-4292-a9a2-34157a3ab292"
-					(reference "J49")
+					(reference "J31")
 					(unit 1)
 				)
